File: Modules/PoE-Ethernet-Si3402-W5500/PoE-Ethernet-Si3402-W5500.kicad_pcb (KiCad board)
At the start: 4 copper layers, 56 x 84 mm, 82 parts, among them J1 ARJM11C7-114-BA-EW2, T1 FA2924-AL, U1 Si3402-B-GMR, U2 VO618A-3X017T, U3 TLV431BCDBZR, U4 W5500, Y1 25.000MHz CL=12pF

Commit message: Apply the review fixes to five boards and set solid power pads
Plans were proven on scratch copies, then applied with KiCad's own pcbnew
Python API, so KiCad writes every file. Each board: DRC 0 errors, 0
unconnected, 0 parity, and the canary fires.

Ethernet and PoE module (R1-1, R1-2, R1-3):
- The fanout rule no longer matches zones.
- Chip-side copper keeps 1.0 mm from the line-side jack pads (was 0.26 mm):
  MDI_RDP, MDI_RDN, RCT and LED_LINK_K rerouted. A 1.0 mm rule enforces it.
  The VC1P lane passes J2.8 at 0.42 mm inside the jack pad field, and only
  that pair is excepted.
- GND vias: Ethernet 8 to 42, PoE 11 to 55. No starved thermal remains.

Buck (R2-2, R2-5): three GND vias at U8.1, C100.2 and C101.2. TP3 sits
against R61.1, with a courtyard rule scoped to that pair.
USBC (R2-4): U2 moves 3 mm toward J1, with two GND vias at U2.2.
MCU (R1-9): C2 sits 1.71 mm from U1 pin 3 (was 23.5 mm), with a courtyard
rule scoped to C2 and U1.
Solid zone connections (R2-3) on U8, L30, C100 to C104, C108 to C111 and J1.

Co-Authored-By: Claude Opus 5.5 (1M context) <noreply@anthropic.com>
Claude-Session: https://claude.ai/code/session_01ErAAfkmF4h3T5yfrw21utF
Routing:
- net /VPOS: track 5.15 -> 8.93 mm
- net GND: track 3.49 -> 7.03 mm, vias 11 -> 55
- net /MDI_RDP: track 23.0 -> 23.8 mm
- net /RCT: track 27.2 -> 27.9 mm
- net /XO: track 11.4 -> 10.8 mm
- net /MDI_RDN: track 19.4 -> 19.9 mm
