File: BlockBuilder/BlockBuilder.kicad_sch (KiCad schematic)
At the start: 82 parts, among them J1 ARJM11C7-114-BA-EW2, T1 FA2924-AL, U1 W5500, U2 Si3402-B-GMR, U3 VO618A-3X017T, U4 TLV431BCDBZR, Y1 25.000MHz CL=12pF

Commit message: Finish the layout blocks: placement tests pass, docs updated
All nine fragments passed the BlockBuilder placement test on 2026-09-25:
footprints, segments, vias, zones and F.Fab labels arrived, and copper
matched each module board net by net. BlockBuilder keeps the PoE retest.

Per-footprint zone-connection overrides do not travel with a fragment. The
Buck, PowerMux and USBC Host-Setup pages say how to set the power pads to
solid in the host.

The PoE module gets its review-fix record (Layout-Spec section 17) and the new
line-side rule in Host-Setup. TODO.md closes the layout block list and lists
the fab questions and known limits. ARCHITECTURE.md carries the new
placement measurement.

Co-Authored-By: Claude Opus 5.5 (1M context) <noreply@anthropic.com>
Claude-Session: https://claude.ai/code/session_01ErAAfkmF4h3T5yfrw21utF
Other:
- moved on the sheet: C1, C10, C11, C12, C13, C14, C15, C16, C17, C18, C19, C2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

Commit message: Put the PoE block schematic on one A3 page
The block schematic spanned 296 mm on an A4 landscape page, and 37 of its 82
parts sat above the frame, so a print lost them.

- Two sheets inside one block do not work: KiCad 10.0.6 refuses to save a
  design block with a nested sheet. Tested on a scratch project.
- The sheet is now A3 portrait with every part inside the frame. Net
  membership is identical to before the move, ERC and DRC are unchanged, and
  the fragment's schematic is updated.
- Placed with Place as sheet, the block lands as its own A3 page with its
  title block. The full layout arrives, copper equal net by net.

Place as sheet prefixes every net with the sheet path, so /NAME net class
patterns bind nothing. Every Host-Setup.md now has section 5.3: use */NAME,
which binds the same nets on a flat placement.

BlockBuilder keeps this test.

Co-Authored-By: Claude Opus 5.5 (1M context) <noreply@anthropic.com>
Claude-Session: https://claude.ai/code/session_01ErAAfkmF4h3T5yfrw21utF
Parts:
- removed C1, C13, C14, C2, C5, C6, C8, C9: 1nF 100V, Capacitor_SMD:C_0603_1608Metric, symbol Device:C
- removed C10, C12, C17, C18, C20, C21, C22, C31: 100nF, Capacitor_SMD:C_0603_1608Metric, symbol Device:C
- removed C11, C16, C7: 1uF 100V, Capacitor_SMD:C_1210_3225Metric, symbol Device:C
- removed C15, C4: 18pF NP0, Capacitor_SMD:C_0603_1608Metric, symbol Device:C
- removed C19: 100nF 100V X7R, Capacitor_SMD:C_1206_3216Metric, symbol Device:C
- removed C23, C34: 10uF 16V, Capacitor_SMD:C_0805_2012Metric, symbol Device:C
- removed C24: 15nF, Capacitor_SMD:C_0603_1608Metric, symbol Device:C
- removed C25, C26: 6.8nF, Capacitor_SMD:C_0603_1608Metric, symbol Device:C
- removed C27: 4.7uF, Capacitor_SMD:C_0805_2012Metric, symbol Device:C
- removed C28, C33: 10nF, Capacitor_SMD:C_0603_1608Metric, symbol Device:C
- removed C29, C30: 1nF Y2 300VAC, Capacitor_THT:C_Disc_D10.5mm_W5.0mm_P10.00mm, symbol Device:C
- removed C3: 33uF 100V, Capacitor_SMD:CP_Elec_10x10.5, symbol Device:C_Polarized
- removed C32: 22nF, Capacitor_SMD:C_0603_1608Metric, symbol Device:C
- removed C35: 3.3nF, Capacitor_SMD:C_0603_1608Metric, symbol Device:C
- removed C36: 470pF 100V C0G, Capacitor_SMD:C_0603_1608Metric, symbol Device:C
- removed C37: 100uF 16V X5R, Capacitor_SMD:C_1210_3225Metric, symbol Device:C
- removed C38: 1000uF 10V, Capacitor_SMD:CP_Elec_10x10.5, symbol Device:C_Polarized
- removed C39: 1nF 2kV, Capacitor_SMD:C_1808_4520Metric, symbol Device:C
- removed D1: 1N4148W, Diode_SMD:D_SOD-123, symbol Device:D
- removed D2: DFLT30A-7, Diode_SMD:D_PowerDI-123, symbol Device:D_Zener
- removed D3: PDS1040-13, Diode_SMD:D_PowerDI-5, symbol Device:D_Schottky
- removed FB1, FB2, FB3, FB4: 330R@100MHz, Inductor_SMD:L_0603_1608Metric, symbol Device:FerriteBead
- removed FB5: 120R@100MHz, Inductor_SMD:L_0603_1608Metric, symbol Device:FerriteBead
- removed J1: ARJM11C7-114-BA-EW2, PoEEthModule:RJ45_Abracon_ARJM11C7-114-BA-EW2, symbol PlumRFBridge:ARJM11C7-114-BA-EW2
- removed L1: 1uH, PoEEthModule:L_Coilcraft_XAL6030, symbol Device:L
- removed R1: 1M, Resistor_SMD:R_0603_1608Metric, symbol Device:R
- removed R10, R12, R23, R5, R7, R8, R9: 0R, Resistor_SMD:R_0603_1608Metric, symbol Device:R
- removed R11: 12.4k 1%, Resistor_SMD:R_0603_1608Metric, symbol Device:R
- removed R13, R14, R15, R16: 49R9 1%, Resistor_SMD:R_0603_1608Metric, symbol Device:R
- removed R17: 10R 1%, Resistor_SMD:R_0603_1608Metric, symbol Device:R
- removed R18: 2.05k, Resistor_SMD:R_0603_1608Metric, symbol Device:R
- removed R19, R20: 330R, Resistor_SMD:R_0603_1608Metric, symbol Device:R
- removed R2: 4.7k, Resistor_SMD:R_0603_1608Metric, symbol Device:R
- removed R21: 36.5k 1%, Resistor_SMD:R_0603_1608Metric, symbol Device:R
- removed R22: 12.1k 1%, Resistor_SMD:R_0603_1608Metric, symbol Device:R
- removed R24: 10R, Resistor_SMD:R_0603_1608Metric, symbol Device:R
- removed R3: 24.3k 1%, Resistor_SMD:R_0603_1608Metric, symbol Device:R
- removed R4: 140R 1%, Resistor_SMD:R_0603_1608Metric, symbol Device:R
- removed R6: 4.99k, Resistor_SMD:R_0603_1608Metric, symbol Device:R
- removed T1: FA2924-AL, PoEEthModule:Transformer_Coilcraft_FA2924-AL, symbol PlumRFBridge:FA2924-AL
- removed TP1: EROUT, TestPoint:TestPoint_Pad_D1.0mm, symbol Connector:TestPoint
- removed TP2: SWO, TestPoint:TestPoint_Pad_D1.0mm, symbol Connector:TestPoint
- removed TP3: VOUT_RAW, TestPoint:TestPoint_Pad_D1.0mm, symbol Connector:TestPoint
- removed U1: W5500, Package_QFP:LQFP-48_7x7mm_P0.5mm, symbol Interface_Ethernet:W5500
- removed U2: Si3402-B-GMR, PoEEthModule:QFN-20-1EP_5x5mm_P0.8mm_EP2.75x2.75mm_Si3402-B, symbol PlumRFBridge:Si3402-B
- removed U3: VO618A-3X017T, Package_DIP:SMDIP-4_W9.53mm_Clearance8mm, symbol Isolator:PC817
- removed U4: TLV431BCDBZR, Package_TO_SOT_SMD:SOT-23, symbol PlumRFBridge:TLV431
- removed Y1: 25.000MHz CL=12pF, Crystal:Crystal_SMD_3225-4Pin_3.2x2.5mm, symbol Device:Crystal_GND24
Connections:
- no-connect marks 18 -> 0
Other:
- added sheet PoE-Ethernet-Si3402-W5500 (PoE-Ethernet-Si3402-W5500.kicad_sch)
- note removed: "100BASE-TX termination: R33/R34 (49R9) bias TD+/TD- to 3V3A and R35 (10R) feeds TCT."
- note removed: "11/12 GREEN. The -AB- part swaps them. Do not substitute. Wave/hand solder only — no reflow part exists."
- note removed: "C57/C58 stay on plain +3V3. Keeping the two apart is what stops SPI noise reaching the PHY."
- note removed: "FB2 splits 3V3A (the W5500's analog/PHY supply) off the digital rail. C50-C56 sit on 3V3A;"
- note removed: "Feedback crosses the barrier optically: U6 senses 5 V through R53/R54 and sinks the U7 LED;"
- note removed: "ISOLATION BARRIER — everything left of the dashed line floats at PoE line potential (up to 57 V)."
- note removed: "J2 LED pins are variant-specific: -BA- is LED Left:Right = Y:G, so 13/14 are YELLOW and"
- note removed: "J2's four line-side centre taps carry PoE to the PD sheet. C67 is the only tie between chassis"
- note removed: "On RX, R36/R37 form the 100 ohm differential load into RCT; C64/C65 AC-couple to the jack."
- note removed: "Only four parts may cross it: T1, the U7 optocoupler, and the C89/C90 3 kV Y-capacitors."
- note removed: "R50 (24.3k) presents the 25k detection signature; R51 (140R) programs Class 1 (<=3.84 W)."
- note removed: "U5 integrates both bridge rectifiers, the detection and classification FETs and the hot-swap switch."
- note removed: "Y1: 25 MHz, CL = 12 pF, +/-30 ppm. R31 (1M) is the bias feedback, R32 (0R) the drive-level trim."
- note removed: "ground (CGND, the RJ45 shell) and signal ground — 1 nF at 2 kV, deliberately not a short."
- note removed: "its phototransistor pulls U5's EROUT pin on the primary side. R56/C86 compensate the loop."
