File: BlockBuilder/PoE-Ethernet-Si3402-W5500.kicad_sch (KiCad schematic)
At the start: 82 parts, among them J1 ARJM11C7-114-BA-EW2, T1 FA2924-AL, U1 Si3402-B-GMR, U2 VO618A-3X017T, U3 TLV431BCDBZR, U4 W5500, Y1 25.000MHz CL=12pF

Commit message: Put the PoE block schematic on one A3 page
The block schematic spanned 296 mm on an A4 landscape page, and 37 of its 82
parts sat above the frame, so a print lost them.

- Two sheets inside one block do not work: KiCad 10.0.6 refuses to save a
  design block with a nested sheet. Tested on a scratch project.
- The sheet is now A3 portrait with every part inside the frame. Net
  membership is identical to before the move, ERC and DRC are unchanged, and
  the fragment's schematic is updated.
- Placed with Place as sheet, the block lands as its own A3 page with its
  title block. The full layout arrives, copper equal net by net.

Place as sheet prefixes every net with the sheet path, so /NAME net class
patterns bind nothing. Every Host-Setup.md now has section 5.3: use */NAME,
which binds the same nets on a flat placement.

BlockBuilder keeps this test.

Co-Authored-By: Claude Opus 5.5 (1M context) <noreply@anthropic.com>
Claude-Session: https://claude.ai/code/session_01ErAAfkmF4h3T5yfrw21utF
Parts:
- renumbered C23 to C10, C9 to C11, C24 to C12, C10 to C13, C11 to C14, C25 to C15, C12 to C16, C26 to C17, C27 to C18, C13 to C19, C14 to C20, C28 to C21, C29 to C22, C30 to C23, C15 to C24, C31 to C25, C32 to C26, C33 to C27, C34 to C28, C16 to C29, C17 to C30, C35 to C31, C36 to C32, C37 to C33, C38 to C34, C18 to C35, C19 to C36, C20 to C37, C21 to C38, C22 to C4, C4 to C5, C5 to C6, C6 to C7, C7 to C8, C8 to C9, R10 to R1, R16 to R10, R17 to R11, R4 to R12, R18 to R13, R19 to R14, R20 to R15, R21 to R16, R22 to R17, R5 to R18, R23 to R19, R11 to R2, R24 to R20, R6 to R21, R7 to R22, R8 to R23, R9 to R24, R1 to R3, R2 to R4, R12 to R5, R3 to R6, R13 to R7, R14 to R8, R15 to R9, U4 to U1, U1 to U2, U2 to U3, U3 to U4
